File: hardware/openScale_v04.brd (EAGLE design)
At the start: 55.9 x 45.7 mm, 69 parts, among them Q1 200mA/50V, Q2 200mA/50V, Q3 MMBT4403, U1 HX711, U3 TMP102, U4 ATMEGA328P_TQFP, U6 FT231XS, Y2 16MHZ

Commit message: Updated Board files
Parts:
- added LOGO1: SFE_LOGO_NAME_FLAME.1_INCH, SparkFun-Aesthetics:SFE_LOGO_NAME_FLAME_.1
- added Q4: MOSFET-NCHANNEL2N7002PW, SparkFun-DiscreteSemi:SOT323
- added R10, R18: 10K, SparkFun-Resistors:0603-RES
- LOGO3: value SFE_LOGO_FLAME.1_STOP -> SFE_LOGO_FLAME.1_INCH; device SparkFun-Aesthetics:SFE_LOGO_FLAME_STOP_.1 -> SparkFun-Aesthetics:SFE_LOGO_FLAME_.1
- S2: device SparkFun-Electromechanical:TACTILE-SWITCH-1101NE -> SparkFun-Electromechanical:TACTILE-SWITCH-SMD
- moved LOGO2 44.6 mm to (24.3, 43.2)
- moved Q1 39.6 mm to (47.9, 10.5)
- moved LOGO3 37.5 mm to (50.5, 5.40)
- moved R9 36.4 mm to (37.8, 10.5)
- moved C3 34.6 mm to (41.6, 11.4), turned to 0 degrees
- moved U3 31.8 mm to (41.6, 9.84)
- moved R8 30.0 mm to (44.8, 10.5)
- moved Q2 29.9 mm to (34.6, 10.5)
- moved C6 29.5 mm to (16.2, 35.6), turned to 270 degrees
- moved C7 29.0 mm to (37.5, 36.5), turned to 90 degrees
- moved R2 27.2 mm to (39.1, 41.9), turned to 180 degrees
- moved D3 23.7 mm to (41.9, 26.4)
- moved C2 23.6 mm to (45.1, 32.4)
- moved R5 23.3 mm to (41.9, 24.1)
- moved D1 23.2 mm to (41.9, 21.9)
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Connections:
- new net N$27: Q4.2, R10.1, U6.1
- new net N$33: Q4.1, R10.2
- net 5V: now also R18.2
- net DTR: now also Q4.3, R18.1; no longer U6.1
- net RST: now also S2.3; no longer S2.2
Routing:
- net 3.3V: track 94.8 -> 50.0 mm, vias 4 -> 0
- net ALERT: track 9.54 -> 53.2 mm, vias 2 -> 8
- net 5V: track 197.7 -> 161.1 mm, vias 9 -> 10
- net GND: track 325.7 -> 296.8 mm, vias 29 -> 36
- net N$14: track 12.1 -> 39.6 mm, vias 2 -> 6
- net RXLED: track 40.7 -> 14.8 mm
- net N$7: track 28.1 -> 3.95 mm
- net TXLED: track 47.3 -> 25.0 mm
- net D13: track 21.5 -> 42.8 mm, vias 1 -> 2
- net RXD: track 34.6 -> 55.2 mm, vias 2 -> 6
- net SDA: track 35.1 -> 54.8 mm
- net N$4: track 21.9 -> 3.93 mm
- net TEMP_DAT: track 49.3 -> 31.4 mm
- net 2: track 12.0 -> 27.4 mm, vias 0 -> 2
- net DTR: track 25.8 -> 39.2 mm
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Other:
- board size 55.9 x 45.7 mm -> 55.9 x 47 mm
