File: hardware/openScale_v04.brd (EAGLE design)
At the start: 55.9 x 47 mm, 73 parts, among them Q1 200mA/50V, Q2 200mA/50V, Q3 MMBT4403, Q4 MOSFET-NCHANNEL2N7002PW, U1 HX711, U3 TMP102, U4 ATMEGA328P_TQFP, U6 FT231XS, Y2 16MHZ

Commit message: Updated Board and Schematic
Parts:
- added LOGO5: OSHW-LOGOS, SparkFun-Aesthetics:OSHW-LOGO-S
- moved LOGO2 43.9 mm to (9.40, 1.91)
Changed lines of the file:
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@@
 <text x="50.6095" y="22.479" size="1.016" layer="22" font="vector" ratio="15" rot="MR90">BLK</text>
 <text x="50.3555" y="9.3345" size="1.016" layer="22" font="vector" ratio="15" rot="MR90">GRN</text>
-<text x="24.8285" y="43.8785" size="1.27" layer="16" font="vector" ratio="15" rot="MR0">v04</text>
+<text x="21.0185" y="44.831" size="1.27" layer="16" font="vector" ratio="15" rot="MR0">v04</text>
 <text x="4.372" y="22.787" size="1.016" layer="21" font="vector" ratio="15" rot="SR270" align="center">BLK
 E-</text>
@@
 <wire x1="13.716" y1="27.94" x2="13.716" y2="10.16" width="0.2032" layer="22"/>
 <wire x1="13.716" y1="10.16" x2="2.54" y2="10.16" width="0.2032" layer="22"/>
-<dimension x1="0" y1="45.72" x2="0" y2="0" x3="-5.08" y3="22.86" textsize="1.778" textratio="15" layer="20" unit="inch"/>
-<dimension x1="55.753" y1="45.72" x2="-0.127" y2="45.72" x3="27.813" y3="51.1175" textsize="1.778" textratio="15" layer="20" unit="inch"/>
+<dimension x1="0" y1="45.72" x2="0" y2="0" x3="-5.08" y3="22.86" textsize="1.778" textratio="15" layer="47" unit="inch"/>
+<dimension x1="55.753" y1="45.72" x2="-0.127" y2="45.72" x3="27.813" y3="51.435" textsize="1.778" textratio="15" layer="47" unit="inch"/>
 <text x="20.193" y="2.794" size="0.8128" layer="21" font="vector" ratio="15">Load Sensor Combinator </text>
 <text x="43.2435" y="2.794" size="0.8128" layer="21" font="vector" ratio="15">3.3V</text>
@@
 <wire x1="0" y1="46.99" x2="55.88" y2="46.99" width="0.2032" layer="20"/>
 <wire x1="55.88" y1="46.99" x2="55.88" y2="45.72" width="0.2032" layer="20"/>
-<text x="62.23" y="43.4975" size="1.778" layer="48" font="vector" ratio="15">All units in Inches</text>
-<dimension x1="2.54" y1="2.54" x2="2.54" y2="42.545" x3="-2.2225" y3="22.5425" textsize="1.778" textratio="15" layer="1" unit="inch"/>
-<dimension x1="2.54" y1="42.545" x2="53.34" y2="42.545" x3="27.94" y3="47.9425" textsize="1.778" textratio="15" layer="1" unit="inch"/>
+<text x="62.23" y="43.4975" size="1.778" layer="51" font="vector" ratio="15">All units in Inches</text>
+<dimension x1="2.54" y1="2.54" x2="2.54" y2="42.545" x3="-2.2225" y3="22.5425" textsize="1.778" textratio="15" layer="47" unit="inch"/>
+<dimension x1="2.54" y1="42.545" x2="53.34" y2="42.545" x3="27.94" y3="47.9425" textsize="1.778" textratio="15" layer="47" unit="inch"/>
 </plain>
 <attributes>
@@
 <attribute name="PROD_ID" value="CAP-00810" x="41.5925" y="11.43" size="1.27" layer="27" font="vector" ratio="15" display="off"/>
 </element>
-<element name="LOGO2" library="SparkFun-Aesthetics" package="OSHW-LOGO-S" value="OSHW-LOGOS" x="24.3205" y="43.18" rot="MR0"/>
+<element name="LOGO2" library="SparkFun-Aesthetics" package="OSHW-LOGO-S" value="OSHW-LOGOS" x="9.398" y="1.905" rot="MR0"/>
 <element name="LOGO4" library="SparkFun-Aesthetics" package="SFE_LOGO_NAME_FLAME_.1" value="SFE_LOGO_NAME_FLAME.1_INCH" x="18.034" y="41.4655" rot="MR0"/>
 <element name="R8" library="SparkFun-Resistors" package="0603-RES" value="4.7K" x="44.7675" y="10.4775" rot="R90">
@@
 </element>
 <element name="LOGO1" library="SparkFun-Aesthetics" package="SFE_LOGO_NAME_FLAME_.1" value="SFE_LOGO_NAME_FLAME.1_INCH" x="5.6515" y="40.1955"/>
+<element name="LOGO5" library="SparkFun-Aesthetics" package="OSHW-LOGO-S" value="OSHW-LOGOS" x="9.398" y="1.905"/>
 </elements>
 <signals>
@@
 </signal>
 </signals>
-<errors>
-</errors>
 </board>
 </drawing>

Commit message: Updated Board and Schematic after reviewing QC checklist
Parts:
- J1: value (none) -> 3.3V
- J2: value (none) -> UL
- J3: value (none) -> UR
- J4: value (none) -> LL
- J5: value (none) -> LR
- JP1: value (none) -> Temp
- JP11: value (none) -> Screw Terminals
- JP2: value (none) -> Fixed Gain 32
- JP3: value (none) -> Load
- moved FID2 1.80 mm to (5.08, 45.1)
- moved LOGO3 1.80 mm to (49.3, 4.13)
- moved JP9 1.27 mm to (54.6, 10.2)
Routing:
- net LC_SCK: track 27.5 -> 31.5 mm
- net TXD: track 45.8 -> 47.1 mm
- net GND: track 296.8 -> 298.1 mm
- net RXD: track 55.2 -> 54.6 mm
- net 5V: track 161.1 -> 161.6 mm
- net DTR: track 39.2 -> 39.7 mm
