File: hardware/openScale_v04.sch (EAGLE design)
At the start: 69 parts, among them Q1 200mA/50V, Q2 200mA/50V, Q3 MMBT4403, U1 HX711, U3 TMP102, U4 ATMEGA328P_TQFP, U6 FT231XS, Y2 16MHZ

Commit message: Updated Board files
Parts:
- added Q4: MOSFET-NCHANNEL2N7002PW, SparkFun-DiscreteSemi:MOSFET-NCHANNEL2N7002PW
- added R10, R18: 10K, SparkFun-Resistors:10KOHM-1/10W-1%(0603)0603
- LOGO3: value SFE_LOGO_FLAME.1_STOP -> SFE_LOGO_FLAME.1_INCH; device SparkFun-Aesthetics:SFE_LOGO_FLAME.1_STOP -> SparkFun-Aesthetics:SFE_LOGO_FLAME.1_INCH
- S2: device SparkFun-Electromechanical:SWITCH-MOMENTARY-2SMD-1101NE -> SparkFun-Electromechanical:SWITCH-MOMENTARY-2SMD
Connections:
- new net N$27: Q4.S, R10.1, U6.!DTR
- new net N$33: Q4.G, R10.2
- net 5V: now also R18.2
- net DTR: now also Q4.D, R18.1; no longer U6.!DTR
Other:
- moved on the sheet: D1, D2, R11, R12, R13, R15

Commit message: Updated Board and Schematic
Other:
- note added: "Revision by: Mary West"
- moved on the sheet: J2, J3, J4, J5

Commit message: Updated Board and Schematic after reviewing QC checklist
Parts:
- J1: value (none) -> 3.3V
- J2: value (none) -> UL
- J3: value (none) -> UR
- J4: value (none) -> LL
- J5: value (none) -> LR
- JP1: value (none) -> Temp
- JP11: value (none) -> Screw Terminals
- JP2: value (none) -> Fixed Gain 32
- JP3: value (none) -> Load
- L1: device SparkFun-Passives:INDUCTOR0805 -> SparkFun-Passives:INDUCTOR0805-IND
Other:
- note removed: "LL"
- note removed: "LR"
- note removed: "Screw Terminals"
- note removed: "UL"
- note removed: "UR"
Changed lines of the file:
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@@
 <part name="GND17" library="SparkFun" deviceset="GND" device=""/>
 <part name="GND19" library="SparkFun" deviceset="GND" device=""/>
-<part name="P+11" library="SparkFun" deviceset="VCC" device="" value="3.3V"/>
+<part name="P+11" library="SparkFun-Aesthetics" deviceset="3.3V" device="" value="3.3V"/>
 <part name="GND21" library="SparkFun" deviceset="GND" device=""/>
 <part name="GND22" library="SparkFun" deviceset="GND" device=""/>
@@
 <part name="U$8" library="SparkFun" deviceset="5V" device=""/>
 <part name="U$9" library="SparkFun" deviceset="5V" device=""/>
-<part name="JP1" library="SparkFun-Connectors" deviceset="M03" device="1X03_NO_SILK"/>
+<part name="JP1" library="SparkFun-Connectors" deviceset="M03" device="1X03_NO_SILK" value="Temp"/>
 <part name="U$16" library="SparkFun" deviceset="5V" device=""/>
 <part name="GND1" library="SparkFun-Aesthetics" deviceset="GND" device=""/>
@@
 <part name="Y2" library="SparkFun-FreqCtrl" deviceset="RESONATOR" device="16MHZ" value="16MHZ"/>
 <part name="SJ2" library="SparkFun-Passives" deviceset="JUMPER-PAD-2-NC_BY_PASTE" device="" value="JUMPER-PAD-2-NC_BY_PASTE"/>
-<part name="JP2" library="SparkFun-Connectors" deviceset="M02" device="PTH"/>
+<part name="JP2" library="SparkFun-Connectors" deviceset="M02" device="PTH" value="Fixed Gain 32"/>
 <part name="C16" library="SparkFun-Capacitors" deviceset="0.1UF-25V(+80/-20%)(0603)" device="" value="0.1uF"/>
 <part name="GND27" library="SparkFun-Aesthetics" deviceset="GND" device=""/>
@@
 <part name="LOGO3" library="SparkFun-Aesthetics" deviceset="SFE_LOGO_FLAME" device=".1_INCH" value="SFE_LOGO_FLAME.1_INCH"/>
 <part name="JP4" library="SparkFun-Connectors" deviceset="M03" device="SCREW_LOCK" value="Screw"/>
-<part name="JP3" library="SparkFun-Connectors" deviceset="M05" device="NO_SILK"/>
-<part name="JP11" library="SparkFun-Connectors" deviceset="M05" device="SCREW"/>
-<part name="L1" library="SparkFun-Passives" deviceset="INDUCTOR" device="0805" value="3.3uH"/>
-<part name="J2" library="SparkFun-Connectors" deviceset="M03" device="PTH"/>
-<part name="J3" library="SparkFun-Connectors" deviceset="M03" device="PTH"/>
-<part name="J4" library="SparkFun-Connectors" deviceset="M03" device="PTH"/>
-<part name="J5" library="SparkFun-Connectors" deviceset="M03" device="PTH"/>
+<part name="JP3" library="SparkFun-Connectors" deviceset="M05" device="NO_SILK" value="Load"/>
+<part name="JP11" library="SparkFun-Connectors" deviceset="M05" device="SCREW" value="Screw Terminals"/>
+<part name="L1" library="SparkFun-Passives" deviceset="INDUCTOR" device="0805-IND" value="3.3uH"/>
+<part name="J2" library="SparkFun-Connectors" deviceset="M03" device="PTH" value="UL"/>
+<part name="J3" library="SparkFun-Connectors" deviceset="M03" device="PTH" value="UR"/>
+<part name="J4" library="SparkFun-Connectors" deviceset="M03" device="PTH" value="LL"/>
+<part name="J5" library="SparkFun-Connectors" deviceset="M03" device="PTH" value="LR"/>
 <part name="U$6" library="SparkFun" deviceset="5V" device=""/>
-<part name="J1" library="SparkFun-Connectors" deviceset="M01" device="PTH"/>
+<part name="J1" library="SparkFun-Connectors" deviceset="M01" device="PTH" value="3.3V"/>
 <part name="JP6" library="SparkFun-Passives" deviceset="JUMPER-PAD-3-2OF3_NC_BY_PASTE" device=""/>
 <part name="Q4" library="SparkFun-DiscreteSemi" deviceset="MOSFET-NCHANNEL" device="2N7002PW"/>
@@
 <text x="15.24" y="254" size="5.08" layer="97">Load Cell Amplifier</text>
 <text x="322.072" y="191.516" size="2.54" layer="97">7-Bit I2C: 0x49</text>
-<text x="23.368" y="195.834" size="1.778" layer="97">Screw
-Terminals</text>
 <text x="27.94" y="218.44" size="1.778" layer="97">Shield</text>
 <text x="142.494" y="102.362" size="1.778" layer="97">Optional External
@@
 <text x="205.74" y="63.5" size="1.778" layer="97" font="vector">WHT</text>
 <text x="205.74" y="60.96" size="1.778" layer="97" font="vector">BLK</text>
-<text x="210.82" y="55.88" size="1.778" layer="97" font="vector">UL</text>
-<text x="233.68" y="50.8" size="1.778" layer="97" font="vector">UR</text>
-<text x="256.54" y="45.72" size="1.778" layer="97">LL</text>
-<text x="281.94" y="40.64" size="1.778" layer="97" font="vector">LR</text>
 <text x="205.74" y="27.94" size="3.81" layer="97">Combine 4 Load sensors to create 1 load cell</text>
 <text x="185.42" y="78.74" size="5.08" layer="97" font="vector">Load Sensor Combiner</text>
@@
 <instance part="GND17" gate="1" x="287.02" y="104.14"/>
 <instance part="GND19" gate="1" x="218.44" y="121.92"/>
-<instance part="P+11" gate="1" x="276.86" y="142.24"/>
+<instance part="P+11" gate="G$1" x="276.86" y="142.24"/>
 <instance part="GND21" gate="1" x="256.54" y="104.14"/>
 <instance part="GND22" gate="1" x="266.7" y="104.14"/>
@@
 <instance part="JP6" gate="G$1" x="180.34" y="228.6" smashed="yes" rot="R270">
 <attribute name="NAME" x="182.88" y="226.441" size="1.778" layer="95"/>
-<attribute name="VALUE" x="154.94" y="234.315" size="1.778" layer="96"/>
 </instance>
 <instance part="Q4" gate="G$1" x="335.28" y="127" smashed="yes" rot="R270"/>
@@
 <wire x1="276.86" y1="121.92" x2="276.86" y2="116.84" width="0.1524" layer="91"/>
 <junction x="276.86" y="121.92"/>
-<pinref part="P+11" gate="1" pin="VCC"/>
+<pinref part="P+11" gate="G$1" pin="3.3V"/>
 <pinref part="C10" gate="G$1" pin="1"/>
 <pinref part="U6" gate="U$1" pin="!RESET"/>
