File: hardware/SparkFun_openScale.sch (EAGLE design)
At the start: 73 parts, among them J1 3.3V, J2 UL, J3 UR, J4 LL, J5 LR, Q1 200mA/50V, Q2 200mA/50V, Q3 MMBT4403, Q4 MOSFET-NCHANNEL2N7002PW, U1 HX711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

Commit message: Update SparkFun_openScale.sch
Updating AVDD equation to be correct
Other:
- note added: "AVDD = VBG(R1+R2)/R2"
- note removed: "AVDD = VBG(R1+R2)/R1"
Changed lines of the file:
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@@
 Serial Interface</text>
 <text x="137.16" y="238.76" size="1.778" layer="96">VBG = 1.25V</text>
-<text x="86.36" y="241.3" size="1.778" layer="96" font="vector">AVDD = VBG(R1+R2)/R1</text>
+<text x="86.36" y="241.3" size="1.778" layer="96" font="vector">AVDD = VBG(R1+R2)/R2</text>
 <text x="421.64" y="7.62" size="2.54" layer="94" font="vector">v10</text>
 <text x="353.568" y="11.43" size="2.54" layer="94" font="vector">N. Seidle</text>
